File: untitled.sch (EAGLE design)
At the start: 65 parts, among them IC1 SIM900, IC2 ST1S10PHR, IC3 SMF05C, IC5 BQ24072, IC6 SIM68R, X1 ST-SMB-H, X2 ST-SMB-H

Commit message: Silkscreen issues solved
Parts:
- L1: device inductor-sumida-cdrh4d18:INDUCTOR-SUMIDA-CDRH4D18 -> CDRH6D38:INDUCTOR-SUMIDA-CDRH4D18
Changed lines of the file:
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@@
 <?xml version="1.0" encoding="utf-8"?>
 <!DOCTYPE eagle SYSTEM "eagle.dtd">
-<eagle version="6.4">
+<eagle version="6.5.0">
 <drawing>
 <settings>
@@
 <setting verticaltext="up"/>
 </settings>
-<grid distance="0.05" unitdist="inch" unit="inch" style="lines" multiple="1" display="no" altdistance="0.01" altunitdist="inch" altunit="inch"/>
+<grid distance="0.1" unitdist="inch" unit="inch" style="lines" multiple="1" display="no" altdistance="0.01" altunitdist="inch" altunit="inch"/>
 <layers>
-<layer number="1" name="Top" color="4" fill="1" visible="no" active="no"/>
-<layer number="16" name="Bottom" color="1" fill="1" visible="no" active="no"/>
-<layer number="17" name="Pads" color="2" fill="1" visible="no" active="no"/>
-<layer number="18" name="Vias" color="2" fill="1" visible="no" active="no"/>
-<layer number="19" name="Unrouted" color="6" fill="1" visible="no" active="no"/>
-<layer number="20" name="Dimension" color="15" fill="1" visible="no" active="no"/>
-<layer number="21" name="tPlace" color="7" fill="1" visible="no" active="no"/>
-<layer number="22" name="bPlace" color="7" fill="1" visible="no" active="no"/>
-<layer number="23" name="tOrigins" color="15" fill="1" visible="no" active="no"/>
-<layer number="24" name="bOrigins" color="15" fill="1" visible="no" active="no"/>
-<layer number="25" name="tNames" color="7" fill="1" visible="no" active="no"/>
-<layer number="26" name="bNames" color="7" fill="1" visible="no" active="no"/>
-<layer number="27" name="tValues" color="7" fill="1" visible="no" active="no"/>
-<layer number="28" name="bValues" color="7" fill="1" visible="no" active="no"/>
+<layer number="1" name="Top" color="4" fill="1" visible="yes" active="no"/>
+<layer number="16" name="Bottom" color="1" fill="1" visible="yes" active="no"/>
+<layer number="17" name="Pads" color="2" fill="1" visible="yes" active="no"/>
+<layer number="18" name="Vias" color="2" fill="1" visible="yes" active="no"/>
+<layer number="19" name="Unrouted" color="6" fill="1" visible="yes" active="no"/>
+<layer number="20" name="Dimension" color="15" fill="1" visible="yes" active="no"/>
+<layer number="21" name="tPlace" color="7" fill="1" visible="yes" active="no"/>
+<layer number="22" name="bPlace" color="7" fill="1" visible="yes" active="no"/>
+<layer number="23" name="tOrigins" color="15" fill="1" visible="yes" active="no"/>
+<layer number="24" name="bOrigins" color="15" fill="1" visible="yes" active="no"/>
+<layer number="25" name="tNames" color="7" fill="1" visible="yes" active="no"/>
+<layer number="26" name="bNames" color="7" fill="1" visible="yes" active="no"/>
+<layer number="27" name="tValues" color="7" fill="1" visible="yes" active="no"/>
+<layer number="28" name="bValues" color="7" fill="1" visible="yes" active="no"/>
 <layer number="29" name="tStop" color="7" fill="3" visible="no" active="no"/>
 <layer number="30" name="bStop" color="7" fill="6" visible="no" active="no"/>
@@
 <layer number="35" name="tGlue" color="7" fill="4" visible="no" active="no"/>
 <layer number="36" name="bGlue" color="7" fill="5" visible="no" active="no"/>
-<layer number="37" name="tTest" color="7" fill="1" visible="no" active="no"/>
-<layer number="38" name="bTest" color="7" fill="1" visible="no" active="no"/>
+<layer number="37" name="tTest" color="7" fill="1" visible="yes" active="no"/>
+<layer number="38" name="bTest" color="7" fill="1" visible="yes" active="no"/>
 <layer number="39" name="tKeepout" color="4" fill="11" visible="no" active="no"/>
 <layer number="40" name="bKeepout" color="1" fill="11" visible="no" active="no"/>
@@
 <layer number="44" name="Drills" color="7" fill="1" visible="no" active="no"/>
 <layer number="45" name="Holes" color="7" fill="1" visible="no" active="no"/>
-<layer number="46" name="Milling" color="3" fill="1" visible="no" active="no"/>
-<layer number="47" name="Measures" color="7" fill="1" visible="no" active="no"/>
-<layer number="48" name="Document" color="7" fill="1" visible="no" active="no"/>
-<layer number="49" name="Reference" color="7" fill="1" visible="no" active="no"/>
-<layer number="50" name="dxf" color="7" fill="1" visible="no" active="no"/>
-<layer number="51" name="tDocu" color="7" fill="1" visible="no" active="no"/>
-<layer number="52" name="bDocu" color="7" fill="1" visible="no" active="no"/>
-<layer number="53" name="tGND_GNDA" color="7" fill="9" visible="no" active="no"/>
-<layer number="54" name="bGND_GNDA" color="1" fill="9" visible="no" active="no"/>
+<layer number="46" name="Milling" color="3" fill="1" visible="yes" active="no"/>
+<layer number="47" name="Measures" color="7" fill="1" visible="yes" active="no"/>
+<layer number="48" name="Document" color="7" fill="1" visible="yes" active="no"/>
+<layer number="49" name="Reference" color="7" fill="1" visible="yes" active="no"/>
+<layer number="50" name="dxf" color="7" fill="1" visible="yes" active="no"/>
+<layer number="51" name="tDocu" color="7" fill="1" visible="yes" active="no"/>
+<layer number="52" name="bDocu" color="7" fill="1" visible="yes" active="no"/>
+<layer number="53" name="tGND_GNDA" color="7" fill="9" visible="yes" active="no"/>
+<layer number="54" name="bGND_GNDA" color="1" fill="9" visible="yes" active="no"/>
 <layer number="91" name="Nets" color="2" fill="1" visible="yes" active="yes"/>
 <layer number="92" name="Busses" color="1" fill="1" visible="yes" active="yes"/>
@@
 <part name="GND4" library="supply1" deviceset="GND" device=""/>
 <part name="GND5" library="supply1" deviceset="GND" device=""/>
-<part name="L1" library="inductor-sumida-cdrh4d18" deviceset="INDUCTOR-SUMIDA-CDRH4D18" device=""/>
+<part name="L1" library="CDRH6D38" deviceset="INDUCTOR-SUMIDA-CDRH4D18" device=""/>
 <part name="R1" library="rcl" deviceset="R-EU_" device="R0805" value="100k"/>
 <part name="R2" library="rcl" deviceset="R-EU_" device="R0805" value="20k"/>

Commit message: small changes
Parts:
- removed IC6: SIM68R, sim68:SIM68R
- added IC4: SIM900, sim900R:SIM900
- C10: value 1u -> 22u
- C11: value 1u -> 100n
- C12: value 4.7u -> (none); device resistor:C-EUC0805 -> rcl:CPOL-EUA/3216-18R
- C13: value 18p -> 100n
- C14: value (none) -> 18p; device rcl:CPOL-EUA/3216-18R -> resistor:C-EUC0805
- C2: value 22u -> 4.7u
- C3: value 4.7u -> 1u
- C4: value 4.7n -> 4.7u
- C7, C8: value 100n -> 1u
- C9: value 1u -> 4.7n
- IC1: value SIM900 -> SIM68R; device sim900R:SIM900 -> sim68:SIM68R
- IC3: value SMF05C -> BQ24072; device smf05c:SMF05C -> TI-bq24075:BQ24072
- IC5: value BQ24072 -> SMF05C; device TI-bq24075:BQ24072 -> smf05c:SMF05C
- JP2: device pinhead:PINHD-1X1 -> pinhead:PINHD-1X3
- JP3: device pinhead:PINHD-1X1 -> pinhead:PINHD-1X2
- JP5, JP6: device pinhead:PINHD-1X2 -> pinhead:PINHD-1X1
- JP7: device pinhead:PINHD-1X3 -> pinhead:PINHD-1X2
- R1: value 100k -> 33
- R10, R8: value 4.7k -> 20k
- R11: value 150 -> 4.7k
- R12: value 22 -> 4.7k
- R13, R14: value 22 -> 47k
- R15: value 47k -> 4.7k
- R16: value 4.7k -> 47k
- R17: value 33 -> 150
- R18: value 150 -> 22
- R19: value 10 -> 22
- R2: value 20k -> 10
- R20: value 20k -> 4.7k
- R21: value 3.3k -> 47k
- R22: value 47k -> 150
- R23: value 4.7k -> 22
- R3: value 1.5k -> 1.8k; device rcl:R-EU_R0603 -> rcl:R-EU_R0805
- R4: value 1.5k -> 3.3k; device rcl:R-EU_R0603 -> rcl:R-EU_R0805
- R5: value 1.2k -> 1.5k
- R6: value 1.8k -> 1.5k; device rcl:R-EU_R0805 -> rcl:R-EU_R0603
- R7: value 47k -> 1.2k; device rcl:R-EU_R0805 -> rcl:R-EU_R0603
- R9: value 47k -> 100k
- renumbered SIM2 to SIM1
Connections:
- removed net N$16 (its old number): LED1.C, VT3.C
- new net N$37: LED3.C, VT3.C
- net +12V: now also C2.1, JP1.2; no longer C3.1, JP8.2
- net +4.8V: now also C10.1, C3.1, C9.1, IC3.IN, JP3.1, R9.2; no longer C2.1, C4.1, C5.1, IC5.IN, JP6.1, R1.2
- net BAT: now also C4.1, IC3.BAT, JP2.3; no longer C6.1, IC5.BAT, JP7.3
- net DBG_RXD: now also IC4G$1.DBG_RXD, JP8.2; no longer IC1G$1.DBG_RXD, JP5.2
- net DBG_TXD: now also IC4G$1.DBG_TXD, JP8.1; no longer IC1G$1.DBG_TXD, JP5.1
- net GND: now also C12.-, C14.2, C4.2, IC1.GND, IC3.EN1, IC3.TMR, IC3.VSS, IC3.^CE, IC4GND@1.GND, IC4GND@11.GND, IC4GND@12.GND, IC4GND@13.GND, IC4GND@14.GND, IC4GND@15.GND, IC4GND@2.GND, IC4GND@3.GND, IC4GND@4.GND, IC4GND@5.GND, IC4GND@6.GND, IC4GND@7.GND, IC4GND@8.GND, IC4GND@9.GND, IC5.2, JP1.1, JP2.1, R10.1, R13.1, R14.1, R16.1, R3.1, R4.1, R8.1; no longer C12.2, C14.-, C9.2, IC1GND@1.GND, IC1GND@11.GND, IC1GND@12.GND, IC1GND@13.GND, IC1GND@14.GND, IC1GND@15.GND, IC1GND@2.GND, IC1GND@3.GND, IC1GND@4.GND, IC1GND@5.GND, IC1GND@6.GND, IC1GND@7.GND, IC1GND@8.GND, IC1GND@9.GND, IC3.2, IC5.EN1, IC5.TMR, IC5.VSS, IC5.^CE, IC6.GND, JP7.1, JP8.1, R15.1, R2.1, R20.1, R22.1, R5.1, R6.1, R9.1
- net N$10: now also IC4G$1.PWRKEY; no longer IC1G$1.PWRKEY
- net N$11: now also R11.1, R13.2; no longer R7.2, R8.1
- net N$12: now also R12.1, R14.2; no longer R10.1, R9.2
- net N$13: now also IC4G$1.RF_ANT, X2.1; no longer IC1G$1.RF_ANT, X1.1
- net N$14: now also IC5.3, R18.1; no longer IC3.3, R12.1
- net N$15: now also IC5.6, R23.2; no longer IC3.6, R14.2
- net N$17: now also C12.+, IC4G$1.VRTC; no longer C14.+, IC1G$1.VRTC
- net N$18: now also IC5.4, R19.1; no longer IC3.4, R13.1
- net N$19: now also R20.1, R21.2, VT4.B; no longer R15.2, R16.1, VT3.B
- net N$2: now also C11.1, IC4G$1.NRESET; no longer C8.1, IC1G$1.NRESET
- net N$20: now also IC4G$1.NETLIGHT\, R20.2; no longer IC1G$1.NETLIGHT\, R16.2
- net N$21: now also IC1.VCC, R1.1; no longer IC6.VCC, R17.1
- net N$22: now also IC1.V_OUT, R2.1; no longer IC6.V_OUT, R19.1
- net N$23: now also C7.1, IC1.V_ANT, R2.2; no longer C11.1, IC6.V_ANT, R19.2
- net N$24: now also IC1.RF_IN, X1.1; no longer IC6.RF_IN, X2.1
- net N$25: now also IC1.TXD1, JP4.1; no longer IC6.TXD1, JP1.1
- net N$26: now also C8.1, IC1.DET_N; no longer C9.1, IC6.DET_N
- net N$27: now also C5.1, IC1.EINT0; no longer C10.1, IC6.EINT0
- net N$28: now also IC1.RXD; no longer IC6.RXD
- net N$29: now also IC1.TXD; no longer IC6.TXD
- net N$3: now also C9.2, R10.2, R9.1; no longer C4.2, R1.1, R2.2
- net N$30: now also IC1.SCL; no longer IC6.SCL
- net N$31: now also IC1.SDA; no longer IC6.SDA
- net N$32: now also IC1.RXD1, JP4.2; no longer IC6.RXD1, JP1.2
- net N$33: now also IC4G$1.SCL; no longer IC1G$1.SCL
- net N$34: now also IC4G$1.SDA; no longer IC1G$1.SDA
- net N$35: now also R15.1, R16.2, VT3.B; no longer R22.2, R23.1, VT4.B
- net N$36: now also LED3.A, R17.2; no longer LED4.A, R11.2
- net N$38: now also IC4G$1.STATUS, R15.2; no longer IC1G$1.STATUS, R23.2
- net N$4: now also LED2.A, R6.1; no longer LED3.A, R4.1
- net N$45: now also LED4.A, R22.2; no longer LED1.A, R18.2
- net N$5: now also IC3.ISET, R7.2, R8.2; no longer IC5.ISET, R20.2, R5.2
- net N$6: now also IC3.ILIM, R3.2, R4.2; no longer IC5.ILIM, R21.2, R6.2
- net N$7: now also LED1.A, R5.2; no longer LED2.A, R3.2
- net N$8: now also IC3.^CHG, LED2.C; no longer IC5.^CHG, LED3.C
- net N$9: now also IC3.^PGOOD, LED1.C; no longer IC5.^PGOOD, LED2.C
- net POWER: now also JP5.1, R11.2; no longer JP2.1, R8.2
- net RESET: now also JP6.1, R12.2; no longer JP3.1, R10.2
- net RXD: now also IC4G$1.RXD, JP7.2; no longer IC1G$1.RXD, JP4.2
- net SIM_CLK: now also IC4G$1.SIM_CLK, R19.2; no longer IC1G$1.SIM_CLK, R13.2
- net SIM_DATA: now also C14.1, IC4G$1.SIM_DATA, R23.1; no longer C13.1, IC1G$1.SIM_DATA, R14.1
- net SIM_PRESENCE: now also IC4G$1.SIM_PRESENCE; no longer IC1G$1.SIM_PRESENCE
- net SIM_RST: now also IC4G$1.SIM_RST, R18.2; no longer IC1G$1.SIM_RST, R12.2
- net SIM_VDD: now also C13.1, IC4G$1.SIM_VDD, IC5.1; no longer C7.1, IC1G$1.SIM_VDD, IC3.1
- net TS: now also IC3.TS, JP2.2; no longer IC5.TS, JP7.2
- net TXD: now also IC4G$1.TXD, JP7.1; no longer IC1G$1.TXD, JP4.1
- net VBAT: now also C6.1, IC3.EN2, IC3.OUT, IC4VBAT@1.VBAT, IC4VBAT@2.VBAT, IC4VBAT@3.VBAT, JP3.2, R1.2, R17.1, R22.1, R5.1, R6.2; no longer C12.1, IC1VBAT@1.VBAT, IC1VBAT@2.VBAT, IC1VBAT@3.VBAT, IC5.EN2, IC5.OUT, JP6.2, R11.1, R17.2, R18.1, R3.1, R4.2
Other:
- moved on the sheet: C10, C11, C13, C2, C3, C4, C5, C6, C7, C8, C9, JP1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

Commit message: New revision
Power supply moved to the top.
IO consolidated
Parts:
- removed JP2: (no value), pinhead:PINHD-1X3
- removed JP5, JP6: (no value), pinhead:PINHD-1X1
- removed JP7, JP8, JP9: (no value), pinhead:PINHD-1X2
- removed SV1, SV2: (no value), con-lstb:MA04-1
- added C15: 22p C0G, resistor:C-EUC0805
- added C16: 47p C0G, resistor:C-EUC0805
- added C17: 100u, rcl:CPOL-EUB/3528-21W
- added FB1: BLM21PG221SN1D, murata-ferrite:BLM21PG221
- added R24: 10k, rcl:R-EU_R0805
- added R25: 0, rcl:R-EU_R0805
- added X3, X4: DG3XX-02-5.0, degson:DG3XX-02-5.0
- C14: value 18p -> 22p
- JP1: device pinhead:PINHD-1X2 -> pinhead:PINHD-2X6
- JP3: device pinhead:PINHD-1X2 -> pinhead:PINHD-2X2
- JP4: device pinhead:PINHD-1X2 -> pinhead:PINHD-1X2ROUND
- R1: value 33 -> 0
Connections:
- removed net N$21: IC1.VCC, R1.1
- removed net N$28: IC1.RXD, SV1.1
- removed net N$29: IC1.TXD, SV1.2
- removed net N$33: IC4G$1.SCL, JP9.1
- removed net N$34: IC4G$1.SDA, JP9.2
- new net GPS_RXD: IC1.RXD, JP3.3, R25.1
- new net GPS_TXD: IC1.TXD, JP3.1, R1.1
- new net SIM_SCL: IC4G$1.SCL, JP1.2
- new net SIM_SDA: IC4G$1.SDA, JP1.4
- new net VBQ: C6.1, FB1.1, IC1.VCC, IC3.EN2, IC3.OUT, R5.1, R6.2
- net +12V: now also X4-1.KL; no longer JP1.2
- net +4.8V: no longer JP3.1
- net BAT: now also X3-2.KL; no longer JP2.3
- net DBG_RXD: now also JP1.3; no longer JP8.2
- net DBG_TXD: now also JP1.1; no longer JP8.1
- net GND: now also C15.2, C16.2, C17.-, JP1.11, JP1.5, JP1.7, JP1.9, R24.1, X3-1.KL, X4-2.KL; no longer JP1.1, JP2.1, SV2.1, SV2.2, SV2.3, SV2.4
- net N$30: now also JP3.2; no longer SV1.3
- net N$31: now also JP3.4; no longer SV1.4
- net POWER: now also JP1.12; no longer JP5.1
- net RESET: now also JP1.6; no longer JP6.1
- net RXD: now also JP1.10, R1.2; no longer JP7.2
- net TS: now also R24.2; no longer JP2.2
- net TXD: now also JP1.8, R25.2; no longer JP7.1
- net VBAT: now also C15.1, C16.1, C17.+, FB1.2; no longer C6.1, IC3.EN2, IC3.OUT, JP3.2, R1.2, R5.1, R6.2
Other:
- moved on the sheet: R1

Commit message: Production ready version
Parts:
- removed JP3: (no value), pinhead:PINHD-2X2
- JP1: device pinhead:PINHD-2X6 -> pinhead:PINHD-2X9
Connections:
- removed net N$30: IC1.SCL, JP3.2
- removed net N$31: IC1.SDA, JP3.4
- new net GPS_SCL: IC1.SCL, JP1.17
- new net GPS_SDA: IC1.SDA, JP1.15
- new net VDD_EXT: IC4G$1.VDD_EXT, JP1.14
- net GND: now also JP1.13
- net GPS_RXD: now also JP1.18; no longer JP3.3
- net GPS_TXD: now also JP1.16; no longer JP3.1
